Commit message: moveit 패키지 이름변경, 작동 확인

File: rh_plus_2_axis_manipulator_description/urdf/materials.xacro (robot description, xacro)
@@ -1,4 +1,4 @@
 <?xml version="1.0" ?>
-<robot name="two_axis_manipulator" xmlns:xacro="http://www.ros.org/wiki/xacro" >
+<robot name="rh_plus_2_axis_manipulator" xmlns:xacro="http://www.ros.org/wiki/xacro" >
 <material name="silver">
   <color rgba="0.700 0.700 0.700 1.000"/>

File: rh_plus_2_axis_manipulator_description/urdf/rh_plus_2_axis_manipulator.xacro (robot description, xacro)
@@ -1,8 +1,8 @@
 <?xml version="1.0" ?>
-<robot name="two_axis_manipulator" xmlns:xacro="http://www.ros.org/wiki/xacro">
-<xacro:include filename="$(find two_axis_manipulator_description)/urdf/materials.xacro" />
-<xacro:include filename="$(find two_axis_manipulator_description)/urdf/two_axis_manipulator.trans" />
-<xacro:include filename="$(find two_axis_manipulator_description)/urdf/two_axis_manipulator.gazebo" />
-<link name="link1">
+<robot name="rh_plus_2_axis_manipulator" xmlns:xacro="http://www.ros.org/wiki/xacro">
+<xacro:include filename="$(find rh_plus_2_axis_manipulator_description)/urdf/materials.xacro" />
+<xacro:include filename="$(find rh_plus_2_axis_manipulator_description)/urdf/rh_plus_2_axis_manipulator.trans" />
+<xacro:include filename="$(find rh_plus_2_axis_manipulator_description)/urdf/rh_plus_2_axis_manipulator.gazebo" />
+<link name="base_link">
   <inertial>
     <origin xyz="-0.028489844749223864 -0.0042819271393418 0.003029979921764912" rpy="0 0 0"/>
@@ -13,5 +13,5 @@
     <origin xyz="0 0 0" rpy="0 0 0"/>
     <geometry>
-      <mesh filename="file://$(find two_axis_manipulator_description)/meshes/link1.stl" scale="0.001 0.001 0.001"/>
+      <mesh filename="file://$(find rh_plus_2_axis_manipulator_description)/meshes/base_link.stl" scale="0.001 0.001 0.001"/>
     </geometry>
     <material name="silver"/>
@@ -20,9 +20,9 @@
     <origin xyz="0 0 0" rpy="0 0 0"/>
     <geometry>
-      <mesh filename="file://$(find two_axis_manipulator_description)/meshes/link1.stl" scale="0.001 0.001 0.001"/>
+      <mesh filename="file://$(find rh_plus_2_axis_manipulator_description)/meshes/base_link.stl" scale="0.001 0.001 0.001"/>
     </geometry>
   </collision>
 </link>
-<link name="link2">
+<link name="link1">
   <inertial>
     <origin xyz="0.025757744162237486 -9.095444257478658e-08 -0.025149867597073286" rpy="0 0 0"/>
@@ -33,5 +33,5 @@
     <origin xyz="0.074 0.109897 -0.0708" rpy="0 0 0"/>
     <geometry>
-      <mesh filename="file://$(find two_axis_manipulator_description)/meshes/link2.stl" scale="0.001 0.001 0.001"/>
+      <mesh filename="file://$(find rh_plus_2_axis_manipulator_description)/meshes/link1.stl" scale="0.001 0.001 0.001"/>
     </geometry>
     <material name="silver"/>
@@ -40,9 +40,9 @@
     <origin xyz="0.074 0.109897 -0.0708" rpy="0 0 0"/>
     <geometry>
-      <mesh filename="file://$(find two_axis_manipulator_description)/meshes/link2.stl" scale="0.001 0.001 0.001"/>
+      <mesh filename="file://$(find rh_plus_2_axis_manipulator_description)/meshes/link1.stl" scale="0.001 0.001 0.001"/>
     </geometry>
   </collision>
 </link>
-<link name="link3">
+<link name="link2">
   <inertial>
     <origin xyz="0.026934734885223178 5.378547984769e-08 -0.025394549004305524" rpy="0 0 0"/>
@@ -53,5 +53,5 @@
     <origin xyz="-0.01612 0.109897 -0.0708" rpy="0 0 0"/>
     <geometry>
-      <mesh filename="file://$(find two_axis_manipulator_description)/meshes/link3.stl" scale="0.001 0.001 0.001"/>
+      <mesh filename="file://$(find rh_plus_2_axis_manipulator_description)/meshes/link2.stl" scale="0.001 0.001 0.001"/>
     </geometry>
     <material name="silver"/>
@@ -60,9 +60,9 @@
     <origin xyz="-0.01612 0.109897 -0.0708" rpy="0 0 0"/>
     <geometry>
-      <mesh filename="file://$(find two_axis_manipulator_description)/meshes/link3.stl" scale="0.001 0.001 0.001"/>
+      <mesh filename="file://$(find rh_plus_2_axis_manipulator_description)/meshes/link2.stl" scale="0.001 0.001 0.001"/>
     </geometry>
   </collision>
 </link>
-<link name="link4">
+<link name="link3">
   <inertial>
     <origin xyz="6.675215935558754e-15 -9.095444264417551e-08 0.02134923455920878" rpy="0 0 0"/>
@@ -73,5 +73,5 @@
     <origin xyz="-0.09594 0.109897 -0.0236" rpy="0 0 0"/>
     <geometry>
-      <mesh filename="file://$(find two_axis_manipulator_description)/meshes/link4.stl" scale="0.001 0.001 0.001"/>
+      <mesh filename="file://$(find rh_plus_2_axis_manipulator_description)/meshes/link3.stl" scale="0.001 0.001 0.001"/>
     </geometry>
     <material name="silver"/>
@@ -80,5 +80,5 @@
     <origin xyz="-0.09594 0.109897 -0.0236" rpy="0 0 0"/>
     <geometry>
-      <mesh filename="file://$(find two_axis_manipulator_description)/meshes/link4.stl" scale="0.001 0.001 0.001"/>
+      <mesh filename="file://$(find rh_plus_2_axis_manipulator_description)/meshes/link3.stl" scale="0.001 0.001 0.001"/>
     </geometry>
   </collision>
@@ -86,6 +86,6 @@
 <joint name="joint1" type="revolute">
   <origin xyz="-0.074 -0.109897 0.0708" rpy="0 0 0"/>
-  <parent link="link1"/>
-  <child link="link2"/>
+  <parent link="base_link"/>
+  <child link="link1"/>
   <axis xyz="0.0 0.0 -1.0"/>
   <limit upper="2.094395" lower="-2.094395" effort="100" velocity="4.8"/>
@@ -93,6 +93,6 @@
 <joint name="joint2" type="revolute">
   <origin xyz="0.09012 0.0 0.0" rpy="0 0 0"/>
-  <parent link="link2"/>
-  <child link="link3"/>
+  <parent link="link1"/>
+  <child link="link2"/>
   <axis xyz="0.0 -0.0 -1.0"/>
   <limit upper="2.094395" lower="-2.094395" effort="100" velocity="4.8"/>
@@ -100,6 +100,6 @@
 <joint name="joint3" type="continuous">
   <origin xyz="0.07982 0.0 -0.0472" rpy="0 0 0"/>
-  <parent link="link3"/>
-  <child link="link4"/>
+  <parent link="link2"/>
+  <child link="link3"/>
   <axis xyz="-0.0 0.0 1.0"/>
 </joint>

File: rh_plus_2_axis_manipulator_moveit_config/config/rh_plus_2_axis_manipulator.ros2_control.xacro (robot description, xacro)
@@ -1,5 +1,5 @@
 <?xml version="1.0"?>
 <robot xmlns:xacro="http://www.ros.org/wiki/xacro">
-    <xacro:macro name="two_axis_manipulator_ros2_control" params="name initial_positions_file">
+    <xacro:macro name="rh_plus_2_axis_manipulator_ros2_control" params="name initial_positions_file">
         <xacro:property name="initial_positions" value="${xacro.load_yaml(initial_positions_file)['initial_positions']}"/>
         <ros2_control name="${name}" type="system">
