Commit message: moveit 원점 수정

File: rh_plus_2_axis_manipulator_description/urdf/rh_plus_2_axis_manipulator.xacro (robot description, xacro)
@@ -6,5 +6,5 @@
 <link name="base_link">
   <inertial>
-    <origin xyz="-0.028489844749223864 -0.0042819271393418 0.003029979921764912" rpy="0 0 0"/>
+    <origin xyz="0.06651015525077507 0.12061516381510062 -0.020570236379403316" rpy="0 0 0"/>
     <mass value="0.6681040624387208"/>
     <inertia ixx="0.00376" iyy="0.005272" izz="0.008817" ixy="-0.000229" iyz="0.000154" ixz="9.6e-05"/>
@@ -26,10 +26,10 @@
 <link name="link1">
   <inertial>
-    <origin xyz="0.025757744162237486 -9.095444257478658e-08 -0.025149867597073286" rpy="0 0 0"/>
+    <origin xyz="0.025757744162237885 4.978656376053436e-16 -0.025150083898241596" rpy="0 0 0"/>
     <mass value="0.10098055947342642"/>
     <inertia ixx="2.5e-05" iyy="9.7e-05" izz="8e-05" ixy="0.0" iyz="-0.0" ixz="-1e-06"/>
   </inertial>
   <visual>
-    <origin xyz="0.074 0.109897 -0.0708" rpy="0 0 0"/>
+    <origin xyz="-0.021 -0.015 -0.0472" rpy="0 0 0"/>
     <geometry>
       <mesh filename="file://$(find rh_plus_2_axis_manipulator_description)/meshes/link1.stl" scale="0.001 0.001 0.001"/>
@@ -38,5 +38,5 @@
   </visual>
   <collision>
-    <origin xyz="0.074 0.109897 -0.0708" rpy="0 0 0"/>
+    <origin xyz="-0.021 -0.015 -0.0472" rpy="0 0 0"/>
     <geometry>
       <mesh filename="file://$(find rh_plus_2_axis_manipulator_description)/meshes/link1.stl" scale="0.001 0.001 0.001"/>
@@ -46,10 +46,10 @@
 <link name="link2">
   <inertial>
-    <origin xyz="0.026934734885223178 5.378547984769e-08 -0.025394549004305524" rpy="0 0 0"/>
+    <origin xyz="0.026934734885221245 1.44739922689624e-07 -0.025394765305473355" rpy="0 0 0"/>
     <mass value="0.10799512775205851"/>
     <inertia ixx="2.4e-05" iyy="9.6e-05" izz="8.2e-05" ixy="-0.0" iyz="0.0" ixz="0.0"/>
   </inertial>
   <visual>
-    <origin xyz="-0.01612 0.109897 -0.0708" rpy="0 0 0"/>
+    <origin xyz="-0.11112 -0.015 -0.0472" rpy="0 0 0"/>
     <geometry>
       <mesh filename="file://$(find rh_plus_2_axis_manipulator_description)/meshes/link2.stl" scale="0.001 0.001 0.001"/>
@@ -58,5 +58,5 @@
   </visual>
   <collision>
-    <origin xyz="-0.01612 0.109897 -0.0708" rpy="0 0 0"/>
+    <origin xyz="-0.11112 -0.015 -0.0472" rpy="0 0 0"/>
     <geometry>
       <mesh filename="file://$(find rh_plus_2_axis_manipulator_description)/meshes/link2.stl" scale="0.001 0.001 0.001"/>
@@ -66,10 +66,10 @@
 <link name="link3">
   <inertial>
-    <origin xyz="6.675215935558754e-15 -9.095444264417551e-08 0.02134923455920878" rpy="0 0 0"/>
+    <origin xyz="1.2212453270876722e-15 3.226585665316861e-16 0.021349018258041263" rpy="0 0 0"/>
     <mass value="0.0038258048079866666"/>
     <inertia ixx="1e-06" iyy="1e-06" izz="0.0" ixy="0.0" iyz="-0.0" ixz="0.0"/>
   </inertial>
   <visual>
-    <origin xyz="-0.09594 0.109897 -0.0236" rpy="0 0 0"/>
+    <origin xyz="-0.19094 -0.015 -0.0" rpy="0 0 0"/>
     <geometry>
       <mesh filename="file://$(find rh_plus_2_axis_manipulator_description)/meshes/link3.stl" scale="0.001 0.001 0.001"/>
@@ -78,5 +78,5 @@
   </visual>
   <collision>
-    <origin xyz="-0.09594 0.109897 -0.0236" rpy="0 0 0"/>
+    <origin xyz="-0.19094 -0.015 -0.0" rpy="0 0 0"/>
     <geometry>
       <mesh filename="file://$(find rh_plus_2_axis_manipulator_description)/meshes/link3.stl" scale="0.001 0.001 0.001"/>
@@ -85,5 +85,5 @@
 </link>
 <joint name="joint1" type="revolute">
-  <origin xyz="-0.074 -0.109897 0.0708" rpy="0 0 0"/>
+  <origin xyz="0.021 0.015 0.0472" rpy="0 0 0"/>
   <parent link="base_link"/>
   <child link="link1"/>
@@ -95,5 +95,5 @@
   <parent link="link1"/>
   <child link="link2"/>
-  <axis xyz="0.0 -0.0 -1.0"/>
+  <axis xyz="0.0 0.0 -1.0"/>
   <limit upper="2.094395" lower="-2.094395" effort="100" velocity="4.8"/>
 </joint>
@@ -102,5 +102,5 @@
   <parent link="link2"/>
   <child link="link3"/>
-  <axis xyz="-0.0 0.0 1.0"/>
+  <axis xyz="-0.0 -0.0 1.0"/>
 </joint>
 </robot>

Commit message: 각속도 수정

File: rh_plus_2_axis_manipulator_description/urdf/rh_plus_2_axis_manipulator.xacro (robot description, xacro)
@@ -89,5 +89,5 @@
   <child link="link1"/>
   <axis xyz="0.0 0.0 -1.0"/>
-  <limit upper="2.094395" lower="-2.094395" effort="100" velocity="4.8"/>
+  <limit upper="2.094395" lower="-2.094395" effort="100" velocity="5.8178"/>
 </joint>
 <joint name="joint2" type="revolute">
@@ -96,5 +96,5 @@
   <child link="link2"/>
   <axis xyz="0.0 0.0 -1.0"/>
-  <limit upper="2.094395" lower="-2.094395" effort="100" velocity="4.8"/>
+  <limit upper="2.094395" lower="-2.094395" effort="100" velocity="5.8178"/>
 </joint>
 <joint name="joint3" type="continuous">

Commit message: description, moveit_config 원점, 세팅 최신화

File: rh_plus_2_axis_manipulator_description/urdf/rh_plus_2_axis_manipulator.xacro (robot description, xacro)
@@ -1,106 +1,107 @@
 <?xml version="1.0" ?>
-<robot name="rh_plus_2_axis_manipulator" xmlns:xacro="http://www.ros.org/wiki/xacro">
-<xacro:include filename="$(find rh_plus_2_axis_manipulator_description)/urdf/materials.xacro" />
-<xacro:include filename="$(find rh_plus_2_axis_manipulator_description)/urdf/rh_plus_2_axis_manipulator.trans" />
-<xacro:include filename="$(find rh_plus_2_axis_manipulator_description)/urdf/rh_plus_2_axis_manipulator.gazebo" />
-<link name="base_link">
-  <inertial>
-    <origin xyz="0.06651015525077507 0.12061516381510062 -0.020570236379403316" rpy="0 0 0"/>
-    <mass value="0.6681040624387208"/>
-    <inertia ixx="0.00376" iyy="0.005272" izz="0.008817" ixy="-0.000229" iyz="0.000154" ixz="9.6e-05"/>
-  </inertial>
-  <visual>
-    <origin xyz="0 0 0" rpy="0 0 0"/>
-    <geometry>
-      <mesh filename="file://$(find rh_plus_2_axis_manipulator_description)/meshes/base_link.stl" scale="0.001 0.001 0.001"/>
-    </geometry>
-    <material name="silver"/>
-  </visual>
-  <collision>
-    <origin xyz="0 0 0" rpy="0 0 0"/>
-    <geometry>
-      <mesh filename="file://$(find rh_plus_2_axis_manipulator_description)/meshes/base_link.stl" scale="0.001 0.001 0.001"/>
-    </geometry>
-  </collision>
-</link>
-<link name="link1">
-  <inertial>
-    <origin xyz="0.025757744162237885 4.978656376053436e-16 -0.025150083898241596" rpy="0 0 0"/>
-    <mass value="0.10098055947342642"/>
-    <inertia ixx="2.5e-05" iyy="9.7e-05" izz="8e-05" ixy="0.0" iyz="-0.0" ixz="-1e-06"/>
-  </inertial>
-  <visual>
-    <origin xyz="-0.021 -0.015 -0.0472" rpy="0 0 0"/>
-    <geometry>
-      <mesh filename="file://$(find rh_plus_2_axis_manipulator_description)/meshes/link1.stl" scale="0.001 0.001 0.001"/>
-    </geometry>
-    <material name="silver"/>
-  </visual>
-  <collision>
-    <origin xyz="-0.021 -0.015 -0.0472" rpy="0 0 0"/>
-    <geometry>
-      <mesh filename="file://$(find rh_plus_2_axis_manipulator_description)/meshes/link1.stl" scale="0.001 0.001 0.001"/>
-    </geometry>
-  </collision>
-</link>
-<link name="link2">
-  <inertial>
-    <origin xyz="0.026934734885221245 1.44739922689624e-07 -0.025394765305473355" rpy="0 0 0"/>
-    <mass value="0.10799512775205851"/>
-    <inertia ixx="2.4e-05" iyy="9.6e-05" izz="8.2e-05" ixy="-0.0" iyz="0.0" ixz="0.0"/>
-  </inertial>
-  <visual>
-    <origin xyz="-0.11112 -0.015 -0.0472" rpy="0 0 0"/>
-    <geometry>
-      <mesh filename="file://$(find rh_plus_2_axis_manipulator_description)/meshes/link2.stl" scale="0.001 0.001 0.001"/>
-    </geometry>
-    <material name="silver"/>
-  </visual>
-  <collision>
-    <origin xyz="-0.11112 -0.015 -0.0472" rpy="0 0 0"/>
-    <geometry>
-      <mesh filename="file://$(find rh_plus_2_axis_manipulator_description)/meshes/link2.stl" scale="0.001 0.001 0.001"/>
-    </geometry>
-  </collision>
-</link>
-<link name="link3">
-  <inertial>
-    <origin xyz="1.2212453270876722e-15 3.226585665316861e-16 0.021349018258041263" rpy="0 0 0"/>
-    <mass value="0.0038258048079866666"/>
-    <inertia ixx="1e-06" iyy="1e-06" izz="0.0" ixy="0.0" iyz="-0.0" ixz="0.0"/>
-  </inertial>
-  <visual>
-    <origin xyz="-0.19094 -0.015 -0.0" rpy="0 0 0"/>
-    <geometry>
-      <mesh filename="file://$(find rh_plus_2_axis_manipulator_description)/meshes/link3.stl" scale="0.001 0.001 0.001"/>
-    </geometry>
-    <material name="silver"/>
-  </visual>
-  <collision>
-    <origin xyz="-0.19094 -0.015 -0.0" rpy="0 0 0"/>
-    <geometry>
-      <mesh filename="file://$(find rh_plus_2_axis_manipulator_description)/meshes/link3.stl" scale="0.001 0.001 0.001"/>
-    </geometry>
-  </collision>
-</link>
-<joint name="joint1" type="revolute">
-  <origin xyz="0.021 0.015 0.0472" rpy="0 0 0"/>
-  <parent link="base_link"/>
-  <child link="link1"/>
-  <axis xyz="0.0 0.0 -1.0"/>
-  <limit upper="2.094395" lower="-2.094395" effort="100" velocity="5.8178"/>
-</joint>
-<joint name="joint2" type="revolute">
-  <origin xyz="0.09012 0.0 0.0" rpy="0 0 0"/>
-  <parent link="link1"/>
-  <child link="link2"/>
-  <axis xyz="0.0 0.0 -1.0"/>
-  <limit upper="2.094395" lower="-2.094395" effort="100" velocity="5.8178"/>
-</joint>
-<joint name="joint3" type="continuous">
-  <origin xyz="0.07982 0.0 -0.0472" rpy="0 0 0"/>
-  <parent link="link2"/>
-  <child link="link3"/>
-  <axis xyz="-0.0 -0.0 1.0"/>
-</joint>
+<robot name="rh_plus_2_axis_manipulator"
+  xmlns:xacro="http://www.ros.org/wiki/xacro">
+  <xacro:include filename="$(find rh_plus_2_axis_manipulator_description)/urdf/materials.xacro" />
+  <xacro:include filename="$(find rh_plus_2_axis_manipulator_description)/urdf/rh_plus_2_axis_manipulator.trans" />
+  <xacro:include filename="$(find rh_plus_2_axis_manipulator_description)/urdf/rh_plus_2_axis_manipulator.gazebo" />
+  <link name="base_link">
+    <inertial>
+      <origin xyz="0.06651015525080728 0.12061516381510094 -0.020570236379403296" rpy="0 0 0"/>
+      <mass value="0.6681040624387203"/>
+      <inertia ixx="0.00376" iyy="0.005272" izz="0.008817" ixy="-0.000229" iyz="0.000154" ixz="9.6e-05"/>
+    </inertial>
+    <visual>
+      <origin xyz="0 0 0" rpy="0 0 0"/>
+      <geometry>
+        <mesh filename="file://$(find rh_plus_2_axis_manipulator_description)/meshes/base_link.stl" scale="0.001 0.001 0.001"/>
+      </geometry>
+      <material name="silver"/>
+    </visual>
+    <collision>
+      <origin xyz="0 0 0" rpy="0 0 0"/>
+      <geometry>
+        <mesh filename="file://$(find rh_plus_2_axis_manipulator_description)/meshes/base_link.stl" scale="0.001 0.001 0.001"/>
+      </geometry>
+    </collision>
+  </link>
+  <link name="link1">
+    <inertial>
+      <origin xyz="0.025757744162237344 7.806255641895632e-17 -0.02515008389824118" rpy="0 0 0"/>
+      <mass value="0.1009805594734264"/>
+      <inertia ixx="2.5e-05" iyy="9.7e-05" izz="8e-05" ixy="-0.0" iyz="-0.0" ixz="-1e-06"/>
+    </inertial>
+    <visual>
+      <origin xyz="-0.021 -0.015 -0.0472" rpy="0 0 0"/>
+      <geometry>
+        <mesh filename="file://$(find rh_plus_2_axis_manipulator_description)/meshes/link1.stl" scale="0.001 0.001 0.001"/>
+      </geometry>
+      <material name="silver"/>
+    </visual>
+    <collision>
+      <origin xyz="-0.021 -0.015 -0.0472" rpy="0 0 0"/>
+      <geometry>
+        <mesh filename="file://$(find rh_plus_2_axis_manipulator_description)/meshes/link1.stl" scale="0.001 0.001 0.001"/>
+      </geometry>
+    </collision>
+  </link>
+  <link name="link2">
+    <inertial>
+      <origin xyz="0.02693702142408899 3.5204052693804666e-10 -0.025394767676016155" rpy="0 0 0"/>
+      <mass value="0.10800020556098276"/>
+      <inertia ixx="2.4e-05" iyy="9.6e-05" izz="8.2e-05" ixy="-0.0" iyz="0.0" ixz="0.0"/>
+    </inertial>
+    <visual>
+      <origin xyz="-0.11112 -0.015 -0.0472" rpy="0 0 0"/>
+      <geometry>
+        <mesh filename="file://$(find rh_plus_2_axis_manipulator_description)/meshes/link2.stl" scale="0.001 0.001 0.001"/>
+      </geometry>
+      <material name="silver"/>
+    </visual>
+    <collision>
+      <origin xyz="-0.11112 -0.015 -0.0472" rpy="0 0 0"/>
+      <geometry>
+        <mesh filename="file://$(find rh_plus_2_axis_manipulator_description)/meshes/link2.stl" scale="0.001 0.001 0.001"/>
+      </geometry>
+    </collision>
+  </link>
+  <link name="link3">
+    <inertial>
+      <origin xyz="5.6343818499726694e-15 1.5612511283791264e-16 0.021349018258040035" rpy="0 0 0"/>
+      <mass value="0.0038258048079866666"/>
+      <inertia ixx="1e-06" iyy="1e-06" izz="0.0" ixy="0.0" iyz="-0.0" ixz="0.0"/>
+    </inertial>
+    <visual>
+      <origin xyz="-0.19094 -0.015 0.0" rpy="0 0 0"/>
+      <geometry>
+        <mesh filename="file://$(find rh_plus_2_axis_manipulator_description)/meshes/link3.stl" scale="0.001 0.001 0.001"/>
+      </geometry>
+      <material name="silver"/>
+    </visual>
+    <collision>
+      <origin xyz="-0.19094 -0.015 0.0" rpy="0 0 0"/>
+      <geometry>
+        <mesh filename="file://$(find rh_plus_2_axis_manipulator_description)/meshes/link3.stl" scale="0.001 0.001 0.001"/>
+      </geometry>
+    </collision>
+  </link>
+  <joint name="joint1" type="revolute">
+    <origin xyz="0.021 0.015 0.0472" rpy="0 0 0"/>
+    <parent link="base_link"/>
+    <child link="link1"/>
+    <axis xyz="0.0 0.0 -1.0"/>
+    <limit upper="2.094395" lower="-2.094395" effort="100" velocity="5.8178"/>
+  </joint>
+  <joint name="joint2" type="revolute">
+    <origin xyz="0.09012 0.0 0.0" rpy="0 0 0"/>
+    <parent link="link1"/>
+    <child link="link2"/>
+    <axis xyz="0.0 0.0 -1.0"/>
+    <limit upper="2.094395" lower="-2.094395" effort="100" velocity="5.8178"/>
+  </joint>
+  <joint name="joint3" type="continuous">
+    <origin xyz="0.07982 0.0 -0.0472" rpy="0 0 0"/>
+    <parent link="link2"/>
+    <child link="link3"/>
+    <axis xyz="0.0 0.0 -1.0"/>
+  </joint>
 </robot>

Commit message: mesh(stl) 파일 원점 제대로 이동

File: rh_plus_2_axis_manipulator_description/urdf/rh_plus_2_axis_manipulator.xacro (robot description, xacro)
@@ -32,5 +32,5 @@
     </inertial>
     <visual>
-      <origin xyz="-0.021 -0.015 -0.0472" rpy="0 0 0"/>
+      <origin xyz="0 0 0" rpy="0 0 0"/>
       <geometry>
         <mesh filename="file://$(find rh_plus_2_axis_manipulator_description)/meshes/link1.stl" scale="0.001 0.001 0.001"/>
@@ -39,5 +39,5 @@
     </visual>
     <collision>
-      <origin xyz="-0.021 -0.015 -0.0472" rpy="0 0 0"/>
+      <origin xyz="0 0 0" rpy="0 0 0"/>
       <geometry>
         <mesh filename="file://$(find rh_plus_2_axis_manipulator_description)/meshes/link1.stl" scale="0.001 0.001 0.001"/>
@@ -52,5 +52,5 @@
     </inertial>
     <visual>
-      <origin xyz="-0.11112 -0.015 -0.0472" rpy="0 0 0"/>
+      <origin xyz="0 0 0" rpy="0 0 0"/>
       <geometry>
         <mesh filename="file://$(find rh_plus_2_axis_manipulator_description)/meshes/link2.stl" scale="0.001 0.001 0.001"/>
@@ -59,5 +59,5 @@
     </visual>
     <collision>
-      <origin xyz="-0.11112 -0.015 -0.0472" rpy="0 0 0"/>
+      <origin xyz="0 0 0" rpy="0 0 0"/>
       <geometry>
         <mesh filename="file://$(find rh_plus_2_axis_manipulator_description)/meshes/link2.stl" scale="0.001 0.001 0.001"/>
@@ -72,5 +72,5 @@
     </inertial>
     <visual>
-      <origin xyz="-0.19094 -0.015 0.0" rpy="0 0 0"/>
+      <origin xyz="0 0 0" rpy="0 0 0"/>
       <geometry>
         <mesh filename="file://$(find rh_plus_2_axis_manipulator_description)/meshes/link3.stl" scale="0.001 0.001 0.001"/>
@@ -79,5 +79,5 @@
     </visual>
     <collision>
-      <origin xyz="-0.19094 -0.015 0.0" rpy="0 0 0"/>
+      <origin xyz="0 0 0" rpy="0 0 0"/>
       <geometry>
         <mesh filename="file://$(find rh_plus_2_axis_manipulator_description)/meshes/link3.stl" scale="0.001 0.001 0.001"/>

Commit message: joint3 제한 걸어주기..!

File: rh_plus_2_axis_manipulator_description/urdf/rh_plus_2_axis_manipulator.xacro (robot description, xacro)
@@ -89,5 +89,5 @@
     <parent link="base_link"/>
     <child link="link1"/>
-    <axis xyz="0.0 0.0 -1.0"/>
+    <axis xyz="0 0 -1"/>
     <limit upper="2.094395" lower="-2.094395" effort="100" velocity="5.8178"/>
   </joint>
@@ -96,12 +96,13 @@
     <parent link="link1"/>
     <child link="link2"/>
-    <axis xyz="0.0 0.0 -1.0"/>
+    <axis xyz="0 0 -1"/>
     <limit upper="2.094395" lower="-2.094395" effort="100" velocity="5.8178"/>
   </joint>
-  <joint name="joint3" type="continuous">
+  <joint name="joint3" type="revolute">
     <origin xyz="0.07982 0.0 -0.0472" rpy="0 0 0"/>
     <parent link="link2"/>
     <child link="link3"/>
-    <axis xyz="0.0 0.0 -1.0"/>
+    <axis xyz="0 0 -1"/>
+    <limit upper="7.0" lower="-7.0" effort="100" velocity="5.8178"/>
   </joint>
 </robot>

Commit message: inertia 관련 에러로 삭제!

File: rh_plus_2_axis_manipulator_description/urdf/rh_plus_2_axis_manipulator.xacro (robot description, xacro)
@@ -6,9 +6,4 @@
   <xacro:include filename="$(find rh_plus_2_axis_manipulator_description)/urdf/rh_plus_2_axis_manipulator.gazebo" />
   <link name="base_link">
-    <inertial>
-      <origin xyz="0.06651015525080728 0.12061516381510094 -0.020570236379403296" rpy="0 0 0"/>
-      <mass value="0.6681040624387203"/>
-      <inertia ixx="0.00376" iyy="0.005272" izz="0.008817" ixy="-0.000229" iyz="0.000154" ixz="9.6e-05"/>
-    </inertial>
     <visual>
       <origin xyz="0 0 0" rpy="0 0 0"/>
@@ -26,9 +21,4 @@
   </link>
   <link name="link1">
-    <inertial>
-      <origin xyz="0.025757744162237344 7.806255641895632e-17 -0.02515008389824118" rpy="0 0 0"/>
-      <mass value="0.1009805594734264"/>
-      <inertia ixx="2.5e-05" iyy="9.7e-05" izz="8e-05" ixy="-0.0" iyz="-0.0" ixz="-1e-06"/>
-    </inertial>
     <visual>
       <origin xyz="0 0 0" rpy="0 0 0"/>
@@ -46,9 +36,4 @@
   </link>
   <link name="link2">
-    <inertial>
-      <origin xyz="0.02693702142408899 3.5204052693804666e-10 -0.025394767676016155" rpy="0 0 0"/>
-      <mass value="0.10800020556098276"/>
-      <inertia ixx="2.4e-05" iyy="9.6e-05" izz="8.2e-05" ixy="-0.0" iyz="0.0" ixz="0.0"/>
-    </inertial>
     <visual>
       <origin xyz="0 0 0" rpy="0 0 0"/>
@@ -66,9 +51,4 @@
   </link>
   <link name="link3">
-    <inertial>
-      <origin xyz="5.6343818499726694e-15 1.5612511283791264e-16 0.021349018258040035" rpy="0 0 0"/>
-      <mass value="0.0038258048079866666"/>
-      <inertia ixx="1e-06" iyy="1e-06" izz="0.0" ixy="0.0" iyz="-0.0" ixz="0.0"/>
-    </inertial>
     <visual>
       <origin xyz="0 0 0" rpy="0 0 0"/>

Commit message: ik solver 변경, position&orientation 수신 에러 해결 완료.

File: rh_plus_2_axis_manipulator_description/urdf/rh_plus_2_axis_manipulator.xacro (robot description, xacro)
@@ -79,10 +79,9 @@
     <limit upper="2.094395" lower="-2.094395" effort="100" velocity="5.8178"/>
   </joint>
-  <joint name="joint3" type="revolute">
+  <joint name="joint3" type="continuous">
     <origin xyz="0.07982 0.0 -0.0472" rpy="0 0 0"/>
     <parent link="link2"/>
     <child link="link3"/>
     <axis xyz="0 0 -1"/>
-    <limit upper="7.0" lower="-7.0" effort="100" velocity="5.8178"/>
   </joint>
 </robot>

Commit message: joint3 전부 제거

File: rh_plus_2_axis_manipulator_description/urdf/rh_plus_2_axis_manipulator.xacro (robot description, xacro)
@@ -50,19 +50,4 @@
     </collision>
   </link>
-  <link name="link3">
-    <visual>
-      <origin xyz="0 0 0" rpy="0 0 0"/>
-      <geometry>
-        <mesh filename="file://$(find rh_plus_2_axis_manipulator_description)/meshes/link3.stl" scale="0.001 0.001 0.001"/>
-      </geometry>
-      <material name="silver"/>
-    </visual>
-    <collision>
-      <origin xyz="0 0 0" rpy="0 0 0"/>
-      <geometry>
-        <mesh filename="file://$(find rh_plus_2_axis_manipulator_description)/meshes/link3.stl" scale="0.001 0.001 0.001"/>
-      </geometry>
-    </collision>
-  </link>
   <joint name="joint1" type="revolute">
     <origin xyz="0.021 0.015 0.0472" rpy="0 0 0"/>
@@ -79,9 +64,3 @@
     <limit upper="2.094395" lower="-2.094395" effort="100" velocity="5.8178"/>
   </joint>
-  <joint name="joint3" type="continuous">
-    <origin xyz="0.07982 0.0 -0.0472" rpy="0 0 0"/>
-    <parent link="link2"/>
-    <child link="link3"/>
-    <axis xyz="0 0 -1"/>
-  </joint>
 </robot>

File: rh_plus_2_axis_manipulator_moveit_config/config/rh_plus_2_axis_manipulator.ros2_control.xacro (robot description, xacro)
@@ -28,10 +28,4 @@
                 </state_interface>
             </joint>
-            <joint name="joint3">
-                <command_interface name="position"/>
-                <state_interface name="position">
-                  <param name="initial_value">${initial_positions['joint3']}</param>
-                </state_interface>
-            </joint>
         </ros2_control>
     </xacro:macro>

File: rh_plus_2_axis_manipulator_moveit_config/config/rh_plus_2_axis_manipulator.urdf.xacro (robot description, xacro)
@@ -2,8 +2,9 @@
 <robot xmlns:xacro="http://www.ros.org/wiki/xacro" name="rh_plus_2_axis_manipulator">
     <xacro:arg name="initial_positions_file" default="initial_positions.yaml" />
+    <xacro:arg name="ros2_control_hardware_type" default="fake" />
     <!-- Import rh_plus_2_axis_manipulator urdf file -->
     <xacro:include filename="$(find rh_plus_2_axis_manipulator_description)/urdf/rh_plus_2_axis_manipulator.xacro" />
     <!-- Import control_xacro -->
     <xacro:include filename="rh_plus_2_axis_manipulator.ros2_control.xacro" />
-    <xacro:rh_plus_2_axis_manipulator_ros2_control name="FakeSystem" initial_positions_file="$(arg initial_positions_file)"/>
+    <xacro:rh_plus_2_axis_manipulator_ros2_control name="TwomaniSystem" initial_positions_file="$(arg initial_positions_file)" ros2_control_hardware_type="$(arg ros2_control_hardware_type)"/>
 </robot>

Commit message: 다시 복구 joint 3 복구

File: rh_plus_2_axis_manipulator_description/urdf/rh_plus_2_axis_manipulator.xacro (robot description, xacro)
@@ -50,4 +50,19 @@
     </collision>
   </link>
+  <link name="link3">
+    <visual>
+      <origin xyz="0 0 0" rpy="0 0 0"/>
+      <geometry>
+        <mesh filename="file://$(find rh_plus_2_axis_manipulator_description)/meshes/link3.stl" scale="0.001 0.001 0.001"/>
+      </geometry>
+      <material name="silver"/>
+    </visual>
+    <collision>
+      <origin xyz="0 0 0" rpy="0 0 0"/>
+      <geometry>
+        <mesh filename="file://$(find rh_plus_2_axis_manipulator_description)/meshes/link3.stl" scale="0.001 0.001 0.001"/>
+      </geometry>
+    </collision>
+  </link>
   <joint name="joint1" type="revolute">
     <origin xyz="0.021 0.015 0.0472" rpy="0 0 0"/>
@@ -64,3 +79,9 @@
     <limit upper="2.094395" lower="-2.094395" effort="100" velocity="5.8178"/>
   </joint>
+  <joint name="joint3" type="continuous">
+    <origin xyz="0.07982 0.0 -0.0472" rpy="0 0 0"/>
+    <parent link="link2"/>
+    <child link="link3"/>
+    <axis xyz="0 0 -1"/>
+  </joint>
 </robot>

File: rh_plus_2_axis_manipulator_moveit_config/config/rh_plus_2_axis_manipulator.ros2_control.xacro (robot description, xacro)
@@ -28,4 +28,10 @@
                 </state_interface>
             </joint>
+            <joint name="joint3">
+                <command_interface name="position"/>
+                <state_interface name="position">
+                  <param name="initial_value">${initial_positions['joint3']}</param>
+                </state_interface>
+            </joint>
         </ros2_control>
     </xacro:macro>
